Commit message: decisao 012: o Livox Mid-360 entra no simulador (raster no lugar da roseta)
Primeira vez que este simulador tem SENSOR. gpu_lidar no topo da caixa,
PointCloud2 em /livox/lidar — mesmo topico do driver real, mesmo principio
do /Odometry. 20 000 pontos/quadro a 10 Hz = 200 000 pontos/s, os numeros
da folha do Mid-360.

O RESULTADO: zona cega de 2,04 m medida (2,20 previsto). Um robo de 45 cm
com ~2 m de cegueira de chao em volta; obstaculo a 1 m so aparece se tiver
mais de 15 cm. E do SENSOR (-7 graus de depressao), nao do simulador, e
nenhuma sintonia de costmap resolve. Para a fatia B sobra memoria ou outro
sensor.

RESSALVA no cabecalho e na decisao: o Mid-360 varre em ROSETA nao
repetitiva e o gpu_lidar varre em RASTER. O simulador enxerga MELHOR num
quadro so. Serve para geometria/zona cega/alcance e para amarrar
nuvem->costmap->Nav2; NAO serve para taxa de deteccao de obstaculo fino
nem para nada sobre FAST-LIO.

A regua errou primeiro, pela terceira vez na semana: a medida saiu 11%
errada porque o script tomava "z minimo" por chao, e z minimo era artefato
de rasancia (pontos 3,8 cm ABAIXO do chao, impossiveis). Virou instrumento
versionado — tools/banco/campo_de_visao.py, puro, 9 testes, um travando
exatamente esse defeito por mutacao.

Junto: a ponte lia <topic> em vez de <topic>/points (subia e nao entregava
nada); junta fixa preservada para a pose do sensor ser conferivel por TF;
e test_massa_total atualizado com os 265 g do Mid-360 — a unica massa do
modelo que vem de folha em vez de chute.

File: ros2_packages/robot_base/description/robo2.gazebo.xacro (robot description, xacro)
@@ -59,3 +59,72 @@
     </plugin>
   </gazebo>
+  <!-- ================= Livox Mid-360, fingido (decisão 012) =================
+       Publica em `/livox/lidar`, o MESMO tópico do driver real — mesmo
+       princípio do `/Odometry`: quem consome não deve saber a diferença.
+       Números da folha do Mid-360: 360° na horizontal, −7° a +52° na
+       vertical, 0,1 a 40 m, 10 Hz, ~200 000 pontos/s (aqui 400×50 = 20 000
+       por quadro a 10 Hz, que dá os mesmos 200 k/s).
+       ⛔ ISTO É RASTER, E O MID-360 É ROSETA NÃO REPETITIVA. Cada quadro
+       real cobre uma FRAÇÃO do campo, e a cobertura adensa com o tempo de
+       integração; aqui a grade é uniforme e igual todo quadro. O simulador
+       portanto ENXERGA MELHOR que o robô num quadro só: obstáculo fino
+       (perna de cadeira) que a roseta pode perder aqui aparece sempre.
+       Serve para: campo de visão, zona cega, alcance, e amarrar a cadeia
+       nuvem→costmap→Nav2. NÃO serve para: taxa de detecção de obstáculo
+       fino, tempo de integração, ou qualquer conclusão sobre FAST-LIO (que
+       se alimenta justamente do padrão de varredura). Racional inteiro e o
+       teste de esparsidade a fazer: `docs/decisoes/012-lidar-3d-no-simulador.md`.
+       ⚠️ A ZONA CEGA É DE PROJETO, não defeito: com −7° de depressão o chão
+       só começa a ~8,1× a altura do sensor. Obstáculo baixo e perto é
+       invisível por geometria, e nenhuma sintonia resolve. -->
+  <!-- ⚠️ A junta fixa TEM de ser preservada. Sem isto o conversor URDF→SDF
+       colapsa `livox_frame` dentro do `base_link` e pendura o sensor lá com
+       a pose remontada — medido em 05-08: o chão aparecia a −0,307 m do
+       sensor quando o modelo diz −0,270, e a zona cega saía inconsistente
+       com o próprio ângulo do feixe (7,7° lidos contra 7,0° configurados).
+       Com a junta preservada a pose do sensor é a que está escrita no URDF,
+       e conferível. Custo: um link a mais na árvore de TF, que é justamente
+       o que a percepção precisa para transformar a nuvem. -->
+  <gazebo reference="livox_joint">
+    <preserveFixedJoint>true</preserveFixedJoint>
+    <disableFixedJointLumping>true</disableFixedJointLumping>
+  </gazebo>
+  <gazebo reference="livox_frame">
+    <sensor name="livox_mid360" type="gpu_lidar">
+      <topic>livox/lidar</topic>
+      <gz_frame_id>livox_frame</gz_frame_id>
+      <update_rate>10</update_rate>
+      <always_on>1</always_on>
+      <visualize>true</visualize>
+      <lidar>
+        <scan>
+          <horizontal>
+            <samples>400</samples>
+            <resolution>1</resolution>
+            <min_angle>-3.141593</min_angle>
+            <max_angle>3.141593</max_angle>
+          </horizontal>
+          <vertical>
+            <samples>50</samples>
+            <resolution>1</resolution>
+            <min_angle>-0.122173</min_angle>  <!-- −7°  -->
+            <max_angle>0.907571</max_angle>   <!-- +52° -->
+          </vertical>
+        </scan>
+        <range>
+          <min>0.1</min>
+          <max>40.0</max>
+          <resolution>0.01</resolution>
+        </range>
+        <!-- ~2 cm é a exatidão de folha do Mid-360. Sem ruído a nuvem sai
+             perfeita e a percepção fica ajustada contra um sensor que não
+             existe — o mesmo erro que a placa fingida existe para não repetir. -->
+        <noise>
+          <type>gaussian</type>
+          <mean>0.0</mean>
+          <stddev>0.02</stddev>
+        </noise>
+      </lidar>
+    </sensor>
+  </gazebo>
 </robot>

File: ros2_packages/robot_base/description/robo2.urdf.xacro (robot description, xacro)
@@ -75,7 +75,17 @@
   <xacro:property name="boba_pivo_atrito"    value="0.05"/>
   <xacro:property name="boba_pivo_damping"   value="0.02"/>
+  <!-- Livox Mid-360, o único sensor externo do robô (decisão 012).
+       ⚠️ POSIÇÃO PROVISÓRIA — mesmo estatuto do `boba_raio`: NÃO medida com
+       trena. Suposto no topo da caixa, centrado. A altura importa muito e é
+       barata de medir: o Mid-360 quase não olha para baixo (−7°), então o
+       chão só aparece a `h/tan(7°) ≈ 8,1·h` do robô. Com estes valores dá
+       um raio cego de ~2,2 m em volta de um robô de 45 cm de largura.
+       Trocar aqui reescala a zona cega inteira. -->
+  <xacro:property name="livox_z_sobre_caixa" value="0.04"/>
+  <xacro:property name="livox_x"             value="0.0"/>
   <!-- ==================== DERIVADOS (não editar) ==================== -->
   <xacro:property name="caixa_cz"  value="${altura_solo + caixa_z/2}"/>
   <xacro:property name="boba_pivo_z" value="${altura_solo}"/>
+  <xacro:property name="livox_z"   value="${altura_solo + caixa_z + livox_z_sobre_caixa}"/>
   <!-- Inércia de caixa sólida.
        ox/oy/oz = onde o CENTRO DE MASSA fica dentro do link. Sem isso o URDF
@@ -180,4 +190,21 @@
     <axis xyz="0 1 0"/>
   </joint>
+  <!-- ==================== Livox Mid-360 (decisão 012) ==================== -->
+  <!-- Corpo cilíndrico de ~65 mm de altura. Sem colisão de propósito: ele não
+       encosta em nada e colisão aqui só criaria contato espúrio no topo. A
+       massa entra porque ele fica ALTO e mexe no centro de massa — 265 g na
+       folha do fabricante. -->
+  <link name="livox_frame">
+    <visual>
+      <geometry><cylinder radius="0.0325" length="0.065"/></geometry>
+      <material name="livox_preto"><color rgba="0.10 0.10 0.12 1"/></material>
+    </visual>
+    <xacro:inercia_roda m="0.265" r="0.0325" h="0.065"/>
+  </link>
+  <joint name="livox_joint" type="fixed">
+    <parent link="base_link"/>
+    <child link="livox_frame"/>
+    <origin xyz="${livox_x} 0 ${livox_z}"/>
+  </joint>
   <!-- ==================== ros2_control ==================== -->
   <!-- Mesmas juntas nos dois casos; só a camada de hardware muda. -->
