Commit message: o robo real ganha corpo: a descricao medida, e o Livox no lugar da trena
Segundo item da fila de dev: destravar o teste D (reflexo de colisao), que
parou na bancada porque NAO EXISTE base_link -> livox_frame no robo.

A MUDANCA E MENOR DO QUE O BLOQUEIO SUGERIA. A arquitetura "uma descricao,
dois hardwares" JA ESTAVA CONSTRUIDA: o robo2.urdf.xacro tem os DOIS blocos
ros2_control (GazeboSimSystem e HoverboardSystem com o plugin real), chaveados
por <xacro:arg name="sim">, e o include do Gazebo esta protegido por xacro:if.
Ela so nunca foi ligada ao robo — o tracao.launch.py carregava o
hoverboard_driver/urdf/diffbot.urdf.xacro, que e o EXEMPLO DE DEMONSTRACAO do
ros2_control:

                  diffbot (o exemplo)      real (trena 29-07)
  caixa           0,10 x 0,10 x 0,05 m    0,433 x 0,455 x 0,145
  raio da roda    0,015 m                  0,080 m
  bitola          0,10 m                   0,270 m
  rodas bobas     duas                     uma
  Livox           nao existe               existe, a 42 cm

Antes de trocar, renderizei os dois xacro e comparei o bloco de hardware:
plugin, juntas, device, wheel_radius, feedback_sign_* e deadband_* saem
IDENTICOS. A troca nao mexe no atuador — muda o corpo.

Verificado subindo o tracao.launch.py aqui, sem placa: "Loaded hardware
'HoverboardSystem'", robot_state_publisher de pe, e a TF base_link ->
livox_frame aparecendo. (O ros2_control_node morre depois, na serial, o que e
esperado sem robo.)

De quebra conserta uma armadilha: o robo2.urdf.xacro traz o comentario "ESTE e
o bloco que o robo le", que era FALSO — e foi essa confusao que fez alguem
editar o arquivo errado em 31-07, segundo o proprio comentario.

ALTURA DO MID-360: 27 cm supostos -> 42 cm MEDIDOS (trena, 05-08)

                    raio cego     a 0,5 m so ve acima de
  suposto (27 cm)    2,19 m              21 cm
  MEDIDO  (42 cm)    3,40 m              36 cm

O simulador estava 55% otimista em zona cega — enxergava obstaculo baixo que o
robo nao enxerga. Consequencia de campo: a caixa do teste D precisa ter 50 cm,
nao os 40 do plano (a 0,5 m sobrariam 4 cm de margem). PLANO_TESTE_ROBO
atualizado.

⚠️ O valor entra DIRETO, sem somar altura_solo nem caixa_z: a medida e do chao
e base_link esta no nivel do chao (a junta da roda fica a roda_raio acima
dele). Somar era o que a versao anterior fazia, e e onde o erro se escondia.

QUATRO TESTES NOVOS, porque nada travava esse numero. O test_urdf_robo2.py
cobria caixa, massa, rodas e boba, e NADA cobria o sensor — a licao de 29-07
("a bancada nao tinha teste nenhum, foi assim que sobreviveu errada").
Entraram: o livox_frame existir na descricao REAL, a altura ser a medida e
centrada, a ZONA CEGA que ela implica (traduz a altura na grandeza que a
operacao sente) e o sensor ser o ponto mais alto do robo. Verificados por
mutacao: voltando aos 27 cm, dois falham.

🔴 ACHADO SEM CONSERTO, e de proposito: o collision_monitor.yaml justifica
max_height: 0.50 dizendo "o robo tem 0,30 m de alto". O robo NAO tem 0,30 m de
alto — a caixa termina a 0,230 e o Mid-360 esta a 0,42. O "0,30" e do modelo
antigo da decisao 004. Nao mexi: max_height e parametro de SEGURANCA e merece
decisao propria, nao efeito colateral desta fatia. Fica travado em teste para
nao passar batido de novo.

517 testes verdes (eram 513).

⚠️ O que SO O ROBO pode confirmar: sessao.py --checar mostrando
wheel_separation = 0.2700 vivo depois da troca de descricao. Primeiro passo da
proxima ida.

File: ros2_packages/robot_base/description/robo2.urdf.xacro (robot description, xacro)
@@ -76,16 +76,28 @@
   <xacro:property name="boba_pivo_damping"   value="0.02"/>
   <!-- Livox Mid-360, o único sensor externo do robô (decisão 012).
-       ⚠️ POSIÇÃO PROVISÓRIA — mesmo estatuto do `boba_raio`: NÃO medida com
-       trena. Suposto no topo da caixa, centrado. A altura importa muito e é
-       barata de medir: o Mid-360 quase não olha para baixo (−7°), então o
-       chão só aparece a `h/tan(7°) ≈ 8,1·h` do robô. Com estes valores dá
-       um raio cego de ~2,2 m em volta de um robô de 45 cm de largura.
-       Trocar aqui reescala a zona cega inteira. -->
-  <xacro:property name="livox_z_sobre_caixa" value="0.04"/>
-  <xacro:property name="livox_x"             value="0.0"/>
+       ✅ MEDIDO COM TRENA em 2026-08-05: centro do sensor a **42 cm do chão**,
+       centrado no robô. Fecha o item que o `ESTADO_PROJETO.md` listava como
+       "o mais barato e de maior retorno da lista".
+       ⚠️ E DERRUBA O QUE ESTAVA AQUI. A posição era suposta (topo da caixa
+       + 4 cm), o que dava 27 cm — **15 cm abaixo do real, 55% de erro**.
+       Como o Mid-360 quase não olha para baixo (−7°), o chão só aparece a
+       `h/tan(7°) ≈ 8,1·h`, e a zona cega escala com a altura:
+           suposto (27 cm)   raio cego 2,19 m   a 0,5 m só vê acima de 21 cm
+           MEDIDO  (42 cm)   raio cego 3,40 m   a 0,5 m só vê acima de 36 cm
+       O simulador estava 55% otimista em zona cega — ele enxergava obstáculo
+       baixo que o robô não enxerga. Consequência de campo: a caixa do teste D
+       precisa ter **50 cm**, não os 40 que o plano pedia (a 0,5 m sobrariam
+       4 cm de margem).
+       ⚠️ A altura é medida DO CHÃO, e `base_link` está no nível do chão (a
+       junta da roda fica a `roda_raio` acima dele). Por isso este valor entra
+       direto, sem somar `altura_solo` nem `caixa_z` — que é o que a versão
+       anterior fazia, e é onde o erro se escondia. -->
+  <xacro:property name="livox_z_solo" value="0.42"/>
+  <xacro:property name="livox_x"      value="0.0"/>
   <!-- ==================== DERIVADOS (não editar) ==================== -->
   <xacro:property name="caixa_cz"  value="${altura_solo + caixa_z/2}"/>
   <xacro:property name="boba_pivo_z" value="${altura_solo}"/>
-  <xacro:property name="livox_z"   value="${altura_solo + caixa_z + livox_z_sobre_caixa}"/>
+  <!-- Medido do chão, e `base_link` está no chão: entra direto. -->
+  <xacro:property name="livox_z"   value="${livox_z_solo}"/>
   <!-- Inércia de caixa sólida.
        ox/oy/oz = onde o CENTRO DE MASSA fica dentro do link. Sem isso o URDF
