Commit message: a D5 fechou olhando o Gazebo: o 37,5 era o EXTERNO, e nada era lixo
O modelo subiu com a bitola 0,425 e o dono olhou: "as rodas estao soltas do
corpo". Depois a frase que resolveu tudo -- "o corpo tem que encostar nas
rodas, pq ele e estreito mesmo esse robo". Essa frase e a medida que faltava, e
ela nao estava em leva nenhuma.

Com o corpo encostando nas rodas, as tres larguras se encaixam sem descartar
nenhuma: lateral da caixa em 12,00, mais o cubo de 1,5 para dentro da 13,50 na
face interna do pneu, mais 5,0 de pneu da 18,50 na externa -- ou seja interno a
interno 27,0, que e o que a 2a leva mediu exato, e externo a externo 37,0
contra os 37,5 da 4a leva. A etiqueta do 37,5 e que estava trocada: ele e o
EXTERNO. E o cubo, cuja resposta "pra dentro do robo" parecia detalhe de
footprint, e exatamente o que preenche o vao. Bitola 0,3225, envelope 0,3725, e
duas rotas independentes concordando em 2,5 mm.

Isso corrige a §5.7 inteira: a bitola cai de 0,425 para 0,3225, o envelope de
0,475 para 0,3725, a folga da porta no pior caso sobe de +6,1 para +10,1 cm por
lado e o teto de giro sobe de 1,46 para 1,93. O C6 volta a ser a boa noticia
que era, agora com todas as medidas usadas em vez de duas descartadas.

A licao de metodo vale para o artigo: a §5.7 escolheu entre duas historias por
argumento -- "o 37,5 foi medido depois da pergunta sem ambiguidade" -- e
escolheu a errada. Quem decidiu nao foi mais discussao, foi DESENHAR E OLHAR.
Nenhuma das duas historias previa que o corpo encosta nas rodas, porque ninguem
tinha perguntado isso; o desenho perguntou sozinho. Fica a regra: medida de
geometria que sobrevive a duas leituras vai para o Gazebo antes de virar
decisao.

As bobas vieram do olho tambem, em duas rodadas, e meu erro nas duas foi
posicionar o PIVO quando a regra e sobre a SUPERFICIE. Agora a face externa da
rodinha e a lateral da caixa e a frente do garfo e a frente da caixa, com recuo
longitudinal ZERO porque o garfo cresce para tras do pivo. O teste passou a
travar alinhamento de faces em vez de distancia escolhida a olho, que ja errou
nos dois sentidos.

E entra a 5.10, a lista para o dono remedir amanha, ordenada por quanto trava.
Com uma regra no topo que teria evitado quatro levas: nunca dizer "centro a
centro" -- medir sempre as DUAS faces e dizer qual e qual, porque o centro se
calcula e a face se mede.

File: ros2_packages/robot_base/description/robo3.urdf.xacro (robot description, xacro)
@@ -48,11 +48,22 @@
   <xacro:property name="altura_solo" value="0.070"/>
   <!-- Motrizes (hoverboard 6,5"). A separação é o divisor do `wz`: errar aqui
-       erra TODO comando de giro, e foi o parâmetro que mais custou a fechar.
-       🟢 DECIDIDO PELO DONO (§5.7): vale a medida de dentro a dentro, 37,5 cm.
-            centro a centro = 37,5 + 5,0 (o pneu) = 42,5 cm
-            envelope        = 37,5 + 2×5,0        = 47,5 cm
-       Os cubos de metal (15 mm) ficam para DENTRO, então quem define a largura
-       do robô é o pneu. Duas outras medidas de largura (27 e 39) foram
-       descartadas por ele; o registro de por quê está na §5.6.1.
+       erra TODO comando de giro, e foi o parâmetro que mais custou a fechar —
+       quatro levas de medida e uma etiqueta trocada.
+       🟢 FECHADO OLHANDO O MODELO NO GAZEBO (§5.9). O dono viu as rodas
+       flutuando longe da caixa e disse o óbvio que nenhuma trena tinha dito:
+       **o corpo encosta nas rodas**. Com essa restrição, TODAS as medidas se
+       encaixam e nenhuma precisa ser descartada:
+           lateral da caixa                 y = 12,00
+           + cubo de metal (para dentro)  1,5 -> face interna do pneu = 13,50
+           + pneu                         5,0 -> face externa do pneu = 18,50
+           interno a interno = 27,0   <- a 2ª leva mediu 27,0    ✅
+           externo a externo = 37,5   <- a 4ª leva mediu 37,5    ✅
+           1ª leva chutou 39,0 de largura total -> 1,5 cm de folga de fita
+       **O CUBO É EXATAMENTE O QUE FECHA O VÃO.** A etiqueta do 37,5 é que
+       estava trocada: ele é o EXTERNO, não o interno. Então:
+           centro a centro = (37,5 + 27,0)/2 = 32,25 cm   <- o valor abaixo
+           envelope        = 32,25 + 5,0     = 37,25 cm
+       Duas rotas independentes concordam em 2,5 mm: a média das duas medidas
+       diretas dá 32,25, e a construção "caixa + cubo + meio pneu" dá 32,00.
        🟢 Raio: diâmetro medido 16,5 cm = 6,5 POLEGADAS EXATAS (6,5 × 2,54 =
        16,51), a roda de hoverboard de catálogo — confirmação independente da
@@ -63,5 +74,9 @@
   <xacro:property name="roda_raio"      value="0.0835"/>
   <xacro:property name="roda_largura"   value="0.050"/>
-  <xacro:property name="roda_separacao" value="0.425"/>
+  <!-- O cubo de metal da roda, 15 mm, virado para DENTRO. Não é decoração: é
+       ele que vence o vão entre a lateral da caixa (y=0,120) e a face interna
+       do pneu (y=0,135), e foi vê-lo faltando no Gazebo que resolveu a D5. -->
+  <xacro:property name="roda_cubo"      value="0.015"/>
+  <xacro:property name="roda_separacao" value="0.3225"/>
   <!-- Onde a caixa fica em relação ao eixo. 🟢 DERIVADO (C5, §5.4.4): dos
        33,1 cm de comprimento total contra 31,1 da caixa sobram 2,0 cm de roda
@@ -85,6 +100,16 @@
   <xacro:property name="boba_raio"  value="0.025"/>
   <xacro:property name="boba_trail" value="0.020"/>
+  <!-- ONDE A BOBA FICA — "as pontas com as pontas" (dono, olhando o Gazebo).
+       A regra NÃO é sobre o pivô, é sobre a SUPERFÍCIE do conjunto: a face
+       externa da rodinha fica rente à lateral da caixa, e a frente do garfo
+       rente à frente da caixa. Duas tentativas erradas antes desta:
+         pivô EM CIMA da quina  -> meia rodinha para fora da lateral
+         pivô recuado 3 cm      -> conjunto boiando longe da borda
+       Então o recuo lateral é meia largura da rodinha, e o longitudinal é
+       ZERO: o garfo cresce para TRÁS do pivô (é o trail), logo a ponta da
+       frente do conjunto É o pivô. -->
+  <xacro:property name="boba_largura" value="0.03"/>
   <xacro:property name="boba_x"     value="${caixa_cx + caixa_x/2}"/>
-  <xacro:property name="boba_y"     value="${caixa_y/2}"/>
+  <xacro:property name="boba_y"     value="${caixa_y/2 - boba_largura/2}"/>
   <!-- ⚠️ MASSAS PROVISÓRIAS — NÃO MEDIDAS.
        O robô ainda não tem Livox nem NUC em cima (D7, §5.4.6), então pesá-lo
@@ -152,8 +177,8 @@
   </link>
   <!-- ==================== MOTRIZES (ATRÁS) ====================
-       Ficam na origem em x, por definição da convenção C8. E ficam FORA da
-       caixa: com o interno em 37,5 e a caixa com 24,0 há 5,25 cm de vão entre
-       a lateral da caixa e cada roda (depois de descontar o cubo). As motrizes
-       estão em balanço, e é por ali que entra pancada lateral. -->
+       Ficam na origem em x, por definição da convenção C8. E ficam ENCOSTADAS
+       na caixa pelo cubo: lateral da caixa em 0,120, cubo até 0,135, pneu de
+       0,135 a 0,185. Zero vão — foi o vão desenhado por engano que denunciou
+       a etiqueta trocada do 37,5. -->
   <xacro:macro name="roda_motriz" params="lado reflect">
     <link name="${lado}_wheel">
@@ -167,4 +192,11 @@
         <geometry><cylinder radius="${roda_raio}" length="${roda_largura}"/></geometry>
       </collision>
+      <!-- O cubo: liga a roda à lateral da caixa. Só visual — quem toca o chão
+           é o pneu, e dar colisão a ele criaria contato lateral que não existe. -->
+      <visual>
+        <origin xyz="0 ${-reflect*(roda_largura+roda_cubo)/2} 0" rpy="${pi/2} 0 0"/>
+        <geometry><cylinder radius="${roda_raio/2}" length="${roda_cubo}"/></geometry>
+        <material name="metal"><color rgba="0.5 0.5 0.55 1"/></material>
+      </visual>
       <xacro:inercia_roda m="${massa_roda}" r="${roda_raio}" h="${roda_largura}"/>
     </link>
@@ -194,8 +226,8 @@
       <visual>
         <origin xyz="${-boba_trail/2} 0 ${-boba_raio/2}"/>
-        <geometry><box size="${boba_trail} 0.03 ${boba_raio}"/></geometry>
+        <geometry><box size="${boba_trail} ${boba_largura} ${boba_raio}"/></geometry>
         <material name="metal"><color rgba="0.5 0.5 0.55 1"/></material>
       </visual>
-      <xacro:inercia_caixa m="${massa_garfo}" x="${boba_trail}" y="0.03" z="${boba_raio}"
+      <xacro:inercia_caixa m="${massa_garfo}" x="${boba_trail}" y="${boba_largura}" z="${boba_raio}"
                            ox="${-boba_trail/2}" oz="${-boba_raio/2}"/>
     </link>
@@ -210,12 +242,12 @@
       <visual>
         <origin rpy="${pi/2} 0 0"/>
-        <geometry><cylinder radius="${boba_raio}" length="0.03"/></geometry>
+        <geometry><cylinder radius="${boba_raio}" length="${boba_largura}"/></geometry>
         <material name="borracha"><color rgba="0.15 0.15 0.15 1"/></material>
       </visual>
       <collision>
         <origin rpy="${pi/2} 0 0"/>
-        <geometry><cylinder radius="${boba_raio}" length="0.03"/></geometry>
+        <geometry><cylinder radius="${boba_raio}" length="${boba_largura}"/></geometry>
       </collision>
-      <xacro:inercia_roda m="${massa_boba}" r="${boba_raio}" h="0.03"/>
+      <xacro:inercia_roda m="${massa_boba}" r="${boba_raio}" h="${boba_largura}"/>
     </link>
     <joint name="${lado}_caster_wheel_joint" type="continuous">

Commit message: a roda e peca de catalogo: 165 mm, 58 mm e 3,1 kg, nao numero de fita
O dono cortou uma linha de trabalho inteira: sao hoverboards genericos de 6,5",
as MESMAS rodas dos robos 1 e 2, e especificacao de peca de catalogo se
pesquisa, nao se mede com fita. Ele esta certo, e eu estava pedindo remedicao
de uma coisa que tem folha de dados.

Hub motor de 6,5": diametro externo 165 mm, largura 58 mm, eixo 45x10, e 3,1 kg
por roda. Os 165 batem com o 16,5 lido no robo 3 e sao 6,5 polegadas exatas; o
perimetro de 53 cm, que daria 16,87, e a fita passando por fora do relevo do
pneu, nao o raio de rolagem. Some a corrida de 5 voltas que eu ia pedir.

O que mais muda e a MASSA, e nao era o que eu estava caçando: 3,1 kg por roda
contra os 2,0 que o robo 2 chutou. As duas rodas sozinhas pesam 6,2 kg, quase o
dobro do chassi, e massa longe do eixo de guinada conta na inercia. O total do
modelo vai de 7,5 para 9,7 kg -- ainda provisorio no chassi, mas com as rodas
agora vindo de folha e nao de palpite.

Raio 0,0825, largura 0,058, envelope 0,3805, teto de giro recalculado para o
patamar 1,903. A porta de 70 fica com +16,0 cm por lado de frente e +9,8 no
pior caso.

O robo 2 fica como esta, com 0,080 e 0,045 nas mesmas rodas: aquele modelo esta
calibrado contra CSV historico e edita-lo retroativamente invalidaria a
comparacao que ele existe para sustentar. Se a diferenca importar, vira linha
no DIARIO.

File: ros2_packages/robot_base/description/robo3.urdf.xacro (robot description, xacro)
@@ -66,12 +66,20 @@
        Duas rotas independentes concordam em 2,5 mm: a média das duas medidas
        diretas dá 32,25, e a construção "caixa + cubo + meio pneu" dá 32,00.
-       🟢 Raio: diâmetro medido 16,5 cm = 6,5 POLEGADAS EXATAS (6,5 × 2,54 =
-       16,51), a roda de hoverboard de catálogo — confirmação independente da
-       trena. O perímetro medido (53 cm) implicaria 16,87, e a diferença de
-       2,2% entre os dois é erro de fita.
-       ⚠️ 0,0835 é o MEIO dos dois, e é PROVISÓRIO: fecha com uma corrida reta
-       de 5 m contra o LIO, onde 2,2% viram 11 cm e ficam óbvios. -->
-  <xacro:property name="roda_raio"      value="0.0835"/>
-  <xacro:property name="roda_largura"   value="0.050"/>
+       🟢 RODA = PEÇA DE CATÁLOGO, e não há o que medir. São hoverboards
+       genéricos de 6,5", as MESMAS rodas dos robôs 1 e 2. Especificação do
+       hub motor de 6,5" (Parallax e fornecedores de peça):
+           diâmetro externo   165 mm   (6,5" = 165,1 mm exatas)
+           largura             58 mm
+           eixo             45 × 10 mm
+           massa              3,1 kg por roda
+       Os 165 mm batem com o 16,5 cm medido no robô 3. O perímetro medido
+       (53 cm) daria 16,87 — 2% a mais, que é a fita passando por FORA do
+       relevo do pneu, não o raio de rolagem.
+       ⚠️ O robô 2 tem 0,080 e 0,045 no URDF dele, medidos com trena em 29-07
+       nas MESMAS rodas. Ficam como estão: aquele modelo está calibrado contra
+       CSV histórico e mexer nele invalidaria a comparação. Se a diferença
+       importar, ela vira uma linha no DIÁRIO, não uma edição retroativa. -->
+  <xacro:property name="roda_raio"      value="0.0825"/>
+  <xacro:property name="roda_largura"   value="0.058"/>
   <!-- O cubo de metal da roda, 15 mm, virado para DENTRO. Não é decoração: é
        ele que vence o vão entre a lateral da caixa (y=0,120) e a face interna
@@ -120,5 +128,9 @@
        de transferência de peso, nem de tombamento deste modelo. -->
   <xacro:property name="massa_chassi" value="3.0"/>
-  <xacro:property name="massa_roda"   value="2.0"/>
+  <!-- 🟢 3,1 kg é de catálogo (Parallax, hub motor 6,5"), não estimativa: o
+       motor mora dentro da roda. O robô 2 usa 2,0 nas MESMAS rodas, e aquilo
+       era chute — aqui as duas rodas sozinhas pesam 6,2 kg, quase o dobro do
+       chassi. É massa longe do eixo de guinada e ela conta. -->
+  <xacro:property name="massa_roda"   value="3.1"/>
   <xacro:property name="massa_garfo"  value="0.05"/>
   <xacro:property name="massa_boba"   value="0.05"/>

Commit message: 17-09: ETAPA 1 fechada -- trena do dono, D3 e D4 encerradas
Quatro valores do URDF corrigidos por medida direta, e NENHUM teste
quebrou (104 passed nos testes do robo 3; suite em 847, so o twist_mux
vendorizado falhando).

  roda_separacao  0,3225 -> 0,320   (38,0 + 26,0)/2
  roda_largura    0,058  -> 0,060   (38,0 - 26,0)/2
  boba_raio       0,025  -> 0,020   chao ate o CENTRO da rodinha = 2,0
  altura_solo     0,070  -> 0,065   topo 20,0 - corpo 13,5

Confirmados sem mexer: caixa 0,311 x 0,240 x 0,135 (o "+-14" fechou em
13,5), topo do corpo 0,200, comprimento do contorno 0,331.

O METODO que deu certo: as duas medidas mais importantes nao foram
lidas direto -- sairam da DIFERENCA entre duas leituras independentes.
Extremo-a-extremo e interna-a-interna dao a bitola pela soma e a
largura da roda pela diferenca. Fita apoiada torto erra as duas para o
mesmo lado e a diferenca cancela. A bitola custou quatro levas de
medida e uma etiqueta trocada; assim fechou de primeira.

BITOLA com TRES caminhos independentes concordando: trena 32,0, desenho
no Gazebo 32,25 (§5.9) e a restricao "o corpo encosta nas rodas".
Espalhamento de 2,5 mm. Os 42,5 da §5.7 morreram de vez, e a
tabela-resumo §5.8 -- que ainda os carregava -- foi corrigida.

D4 NUNCA FOI CAIMENTO, era numero errado. O modelo inventava um
"suporte de 10 mm" sob a boba para acomodar 1 cm de diferenca entre
duas fitas. Topo 20,0 - corpo 13,5 = fundo 6,5, que e exatamente o
"6,5 da boba ate o corpo" medido. Dono: "esta sim alinhado, nao esta
caido nao". Uma hipotese mecanica inteira existia so por causa de um
valor errado.

D3 encerrada pelo mesmo tipo de medida: com a rodinha apoiada, a altura
do centro E o raio. O empate 40 x 50 mm da §5.5.1 acabou.

PLACA RESPONDIDA (§5.1, o item de maior alavancagem): "mesmo modelo do
1 e do 2, mas nao a mesma, cada um tem a sua". Saida boa -- o modelo de
atuador sobrevive e a etapa 8 vira CONFERENCIA, nao levantamento novo.
Ressalva registrada: mesma classe, peca diferente, entao os numeros do
MODELO_ROBO2 sao ponto de partida e nao medida deste robo.

Acompanham: bitola nova nos tres lugares presos ao URDF por teste
(YAML do controlador, sim_robo3, controle_robo3), e o robo3.zip no
.gitignore -- ele estava na raiz nao rastreado e o proximo git add -A
teria posto 2,7 MB de foto no historico.

File: ros2_packages/robot_base/description/robo3.urdf.xacro (robot description, xacro)
@@ -39,12 +39,19 @@
        ⚠️ D4 ABERTA: a boba com estrutura mede 60 mm e o fundo da caixa está a
        70 mm. Se os dois estiverem certos, o robô fica 2,3° caído para a frente
-       ao longo do entre-eixos. Aqui o modelo assume NIVELADO (a boba sobe num
-       suporte de 10 mm), porque inclinação permanente é afirmação forte para
-       sair de uma diferença de 1 cm entre duas medidas de fita. Se a medida
-       com nível confirmar o caimento, ele entra aqui e não em outro lugar. -->
+       ao longo do entre-eixos.
+       🟢 D4 ENCERRADA EM 17-09, e não havia caimento nenhum — havia um número
+       errado. A trena do dono fecha sozinha:
+            topo do corpo    20,0
+            altura do corpo  13,5   −
+                             ─────
+            fundo do corpo    6,5   = os "6,5 da boba até o corpo" medidos
+       Ou seja `altura_solo` é 0,065, e o 0,070 é que estava errado. Palavra do
+       dono: *"ele está sim alinhado, não está caído não"*. Some o suporte de
+       10 mm inventado para explicar a diferença: ela não existia. -->
   <xacro:property name="caixa_x"     value="0.311"/>
   <xacro:property name="caixa_y"     value="0.240"/>
+  <!-- 13,5 confirmado em 17-09 (o dono deu "±14" e fechou em 13,5). -->
   <xacro:property name="caixa_z"     value="0.135"/>
-  <xacro:property name="altura_solo" value="0.070"/>
+  <xacro:property name="altura_solo" value="0.065"/>
   <!-- Motrizes (hoverboard 6,5"). A separação é o divisor do `wz`: errar aqui
        erra TODO comando de giro, e foi o parâmetro que mais custou a fechar —
@@ -81,10 +88,21 @@
        importar, ela vira uma linha no DIÁRIO, não uma edição retroativa. -->
   <xacro:property name="roda_raio"      value="0.0825"/>
-  <xacro:property name="roda_largura"   value="0.058"/>
+  <!-- 🟢 MEDIDO EM 17-09, e sem fita atravessada: o dono deu extremo-a-extremo
+       38,0 e face-interna-a-face-interna 26,0. A largura sai da diferença, que
+       é medida derivada de duas leituras independentes e não de uma fita
+       apoiada torto:  (38,0 − 26,0)/2 = 6,0 cm.
+       Era 0,058 (catálogo) e a tabela §5.8 dizia 0,050 — as duas caem. -->
+  <xacro:property name="roda_largura"   value="0.060"/>
   <!-- O cubo de metal da roda, 15 mm, virado para DENTRO. Não é decoração: é
        ele que vence o vão entre a lateral da caixa (y=0,120) e a face interna
        do pneu (y=0,135), e foi vê-lo faltando no Gazebo que resolveu a D5. -->
   <xacro:property name="roda_cubo"      value="0.015"/>
-  <xacro:property name="roda_separacao" value="0.3225"/>
+  <!-- 🟢 MEDIDA DIRETA EM 17-09, e ela fecha a história:
+            centro a centro = (38,0 + 26,0)/2 = 32,0 cm
+       Bate com os 32,25 que a §5.9 tinha fechado desenhando no Gazebo (2,5 mm
+       de erro de trena) e ENTERRA de vez os 42,5 da §5.7, que a tabela-resumo
+       ainda carregava. Três caminhos independentes — trena, desenho e a
+       restrição "o corpo encosta nas rodas" — dão o mesmo número. -->
+  <xacro:property name="roda_separacao" value="0.320"/>
   <!-- Onde a caixa fica em relação ao eixo. 🟢 DERIVADO (C5, §5.4.4): dos
        33,1 cm de comprimento total contra 31,1 da caixa sobram 2,0 cm de roda
@@ -97,8 +115,11 @@
        🟢 MEDIDO: trail 20 mm, e elas ficam "cada uma na ponta da frente da
        caixa, uma em cada extremidade".
-       🟡 Raio 25 mm ADOTADO: as medidas empataram 2 a 2 entre 40 e 50 mm de
-       diâmetro (§5.5.1). Ficou 50 mm por ser tamanho de catálogo, e o empate
-       é irrelevante porque a altura da frente vem do CONJUNTO (60 mm medidos),
-       não do diâmetro da roda.
+       🟢 RAIO 20 mm MEDIDO EM 17-09 — o empate da §5.5.1 (40 contra 50 mm de
+       diâmetro) acabou, e ganhou o 40: o dono mediu **chão até o centro da
+       rodinha = 2,0 cm**, e com ela apoiada no chão essa altura É o raio.
+       Estava 0,025 aqui, adotado por ser tamanho de catálogo.
+       O conjunto continua tocando o chão, e é o que o modelo garante sozinho:
+       pivô em `altura_solo` 0,065, junta da roda em −(0,065 − 0,020) = −0,045,
+       centro da rodinha em 0,020 = o raio.
        🔴 O TRAIL DOBROU E DUPLICOU (C7, §5.6.3): o robô 2 tinha 10 mm em UMA
        boba, este tem 20 mm em DUAS. Numa inversão de marcha cada boba gira
@@ -106,5 +127,5 @@
        Com o entre-eixos de 24,85 cm isso é até 9,1° de perturbação de rumo
        contra 4,6° — e o robô 2 dava SETE rés numa aproximação de porta. -->
-  <xacro:property name="boba_raio"  value="0.025"/>
+  <xacro:property name="boba_raio"  value="0.020"/>
   <xacro:property name="boba_trail" value="0.020"/>
   <!-- ONDE A BOBA FICA — "as pontas com as pontas" (dono, olhando o Gazebo).
